Commit message: update collision

File: mycobot_description/urdf/mycobot_320_m5_2020/mycobot_pro_320_m5_2020_gripper.urdf (robot description, URDF)
Before this commit: robot firefighter, 15 links, 14 joints
Links:
- link base: geometry visual mesh filename=package://mycobot_description/urdf/mycobot_320_m5_2020/base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
- link gripper_right3: geometry visual mesh filename=package://mycobot_description/urdf/mycobot_320_m5_2020/grip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
